Commit message: fixing

File: description/my_robot.urdf.xacro (robot description, xacro)
@@ -8,5 +8,5 @@
   <xacro:property name="upper_limit" value="6.28"/>
   <xacro:property name="velocity_limit" value="1.0"/>
-  <xacro:property name="effort_limit" value="1000.0"/>
+  <xacro:property name="effort_limit" value="10.0"/>
   <!-- materials -->
   <xacro:include filename="materials.xml"/>
@@ -76,5 +76,5 @@
     </inertial>
   </link>
-  <link name="link3">
+  <!--link name="link3">
     <visual>
       <geometry>
@@ -96,5 +96,5 @@
     </inertial>
   </link>
-  <!--link name="link4">
+  <link name="link4">
     <visual>
       <geometry>
@@ -164,4 +164,5 @@
     <axis xyz="0 0 1"/>
     <limit lower="${lower_limit}" upper="${upper_limit}" velocity="${velocity_limit}" effort="${effort_limit}"/>
+    <dynamics damping="0.7" friction="10.0"/>
   </joint>
   <joint name="joint2" type="revolute">
@@ -171,6 +172,7 @@
     <axis xyz="0 0 1"/>
     <limit lower="${lower_limit}" upper="${upper_limit}" velocity="${velocity_limit}" effort="${effort_limit}"/>
-  </joint>
-  <joint name="joint3" type="revolute">
+    <dynamics damping="0.7" friction="10.0"/>
+  </joint>
+  <!--joint name="joint3" type="revolute">
     <parent link="link2"/>
     <child link="link3"/>
@@ -178,6 +180,7 @@
     <axis xyz="0 0 1"/>
     <limit lower="${lower_limit}" upper="${upper_limit}" velocity="${velocity_limit}" effort="${effort_limit}"/>
-  </joint>
-  <!--joint name="joint4" type="revolute">
+    <dynamics damping="0.7" friction="10.0"/>
+  </joint>
+  <joint name="joint4" type="revolute">
     <parent link="link3"/>
     <child link="link4"/>
