Commit message: update

File: description/my_robot.urdf (robot description, URDF)
Before this commit: robot my_robot, 8 links, 7 joints
Links:
- link link2: geometry collision box size=0.8 0.05 0.05; visual box size=0.8 0.05 0.05
- link link3: geometry collision box size=0.55 0.05 0.05; visual box size=0.55 0.05 0.05
Joints:
- joint joint1: limit lower=${lower_limit} upper=${upper_limit} effort=${effort_limit} velocity=${velocity_limit} -> lower=-3.14 upper=3.14 effort=1000.0 velocity=1.0
- joint joint2: limit lower=${lower_limit} upper=${upper_limit} effort=${effort_limit} velocity=${velocity_limit} -> lower=-3.14 upper=3.14 effort=1000.0 velocity=1.0
- joint joint3: limit lower=${lower_limit} upper=${upper_limit} effort=${effort_limit} velocity=${velocity_limit} -> lower=-3.14 upper=3.14 effort=1000.0 velocity=1.0; origin xyz=${l1} 0 0 rpy=0 0 0 -> xyz=0.75 0 0 rpy=0 0 0
- joint joint4: limit lower=${lower_limit} upper=${upper_limit} effort=${effort_limit} velocity=${velocity_limit} -> lower=-3.14 upper=3.14 effort=1000.0 velocity=1.0; origin xyz=${l2} 0 0 rpy=0 0 0 -> xyz=0.5 0 0 rpy=0 0 0
- joint joint5: limit lower=${lower_limit} upper=${upper_limit} effort=${effort_limit} velocity=${velocity_limit} -> lower=-3.14 upper=3.14 effort=1000.0 velocity=1.0
- joint joint6: limit lower=${lower_limit} upper=${upper_limit} effort=${effort_limit} velocity=${velocity_limit} -> lower=-3.14 upper=3.14 effort=1000.0 velocity=1.0
